File: limit_switch.kicad_sch (KiCad schematic)
At the start: 32 parts

Commit message: 回路図だいたい完成
Parts:
- gave numbers to parts that had none: 32

Commit message: 何こっち見てんだよ
Parts:
- J10: renamed from J21; footprint (none) -> Connector_JST:JST_XH_B2B-XH-A_1x02_P2.50mm_Vertical
- J11: renamed from J22; footprint (none) -> Connector_JST:JST_XH_B2B-XH-A_1x02_P2.50mm_Vertical
- J12: renamed from J23; footprint (none) -> Connector_JST:JST_XH_B2B-XH-A_1x02_P2.50mm_Vertical
- J13: renamed from J24; footprint (none) -> Connector_JST:JST_XH_B2B-XH-A_1x02_P2.50mm_Vertical
- J14: renamed from J25; footprint (none) -> Connector_JST:JST_XH_B2B-XH-A_1x02_P2.50mm_Vertical
- J15: renamed from J26; footprint (none) -> Connector_JST:JST_XH_B2B-XH-A_1x02_P2.50mm_Vertical
- J16: renamed from J27; footprint (none) -> Connector_JST:JST_XH_B2B-XH-A_1x02_P2.50mm_Vertical
- J17: renamed from J28; footprint (none) -> Connector_JST:JST_XH_B2B-XH-A_1x02_P2.50mm_Vertical
- J18: renamed from J29; footprint (none) -> Connector_JST:JST_XH_B2B-XH-A_1x02_P2.50mm_Vertical
- J19: renamed from J30; footprint (none) -> Connector_JST:JST_XH_B2B-XH-A_1x02_P2.50mm_Vertical
- J20: renamed from J31; footprint (none) -> Connector_JST:JST_XH_B2B-XH-A_1x02_P2.50mm_Vertical
- J21: renamed from J32; footprint (none) -> Connector_JST:JST_XH_B2B-XH-A_1x02_P2.50mm_Vertical
- J22: renamed from J33; footprint (none) -> Connector_JST:JST_XH_B2B-XH-A_1x02_P2.50mm_Vertical
- J7: renamed from J18; footprint (none) -> Connector_JST:JST_XH_B2B-XH-A_1x02_P2.50mm_Vertical
- J8: renamed from J19; footprint (none) -> Connector_JST:JST_XH_B2B-XH-A_1x02_P2.50mm_Vertical
- J9: renamed from J20; footprint (none) -> Connector_JST:JST_XH_B2B-XH-A_1x02_P2.50mm_Vertical
- renumbered R9 to R10, R10 to R11, R11 to R12, R12 to R13, R13 to R14, R14 to R15, R15 to R16, R16 to R17, R17 to R18, R18 to R19, R19 to R20, R20 to R21, R21 to R22, R22 to R23, R23 to R24, R8 to R9

Commit message: 配線だいたい完了
Parts:
- removed J10: LIMIT_13, Connector_JST:JST_XH_B2B-XH-A_1x02_P2.50mm_Vertical, symbol Connector:Conn_01x02_Socket
- removed J11: LIMIT_2, Connector_JST:JST_XH_B2B-XH-A_1x02_P2.50mm_Vertical, symbol Connector:Conn_01x02_Socket
- removed J12: LIMIT_6, Connector_JST:JST_XH_B2B-XH-A_1x02_P2.50mm_Vertical, symbol Connector:Conn_01x02_Socket
- removed J13: LIMIT_10, Connector_JST:JST_XH_B2B-XH-A_1x02_P2.50mm_Vertical, symbol Connector:Conn_01x02_Socket
- removed J14: LIMIT_14, Connector_JST:JST_XH_B2B-XH-A_1x02_P2.50mm_Vertical, symbol Connector:Conn_01x02_Socket
- removed J15: LIMIT_3, Connector_JST:JST_XH_B2B-XH-A_1x02_P2.50mm_Vertical, symbol Connector:Conn_01x02_Socket
- removed J16: LIMIT_7, Connector_JST:JST_XH_B2B-XH-A_1x02_P2.50mm_Vertical, symbol Connector:Conn_01x02_Socket
- removed J17: LIMIT_11, Connector_JST:JST_XH_B2B-XH-A_1x02_P2.50mm_Vertical, symbol Connector:Conn_01x02_Socket
- removed J18: LIMIT_15, Connector_JST:JST_XH_B2B-XH-A_1x02_P2.50mm_Vertical, symbol Connector:Conn_01x02_Socket
- removed J19: LIMIT_4, Connector_JST:JST_XH_B2B-XH-A_1x02_P2.50mm_Vertical, symbol Connector:Conn_01x02_Socket
- removed J20: LIMIT_8, Connector_JST:JST_XH_B2B-XH-A_1x02_P2.50mm_Vertical, symbol Connector:Conn_01x02_Socket
- removed J21: LIMIT_12, Connector_JST:JST_XH_B2B-XH-A_1x02_P2.50mm_Vertical, symbol Connector:Conn_01x02_Socket
- removed J22: LIMIT_16, Connector_JST:JST_XH_B2B-XH-A_1x02_P2.50mm_Vertical, symbol Connector:Conn_01x02_Socket
- removed J7: LIMIT_1, Connector_JST:JST_XH_B2B-XH-A_1x02_P2.50mm_Vertical, symbol Connector:Conn_01x02_Socket
- removed J8: LIMIT_5, Connector_JST:JST_XH_B2B-XH-A_1x02_P2.50mm_Vertical, symbol Connector:Conn_01x02_Socket
- removed J9: LIMIT_9, Connector_JST:JST_XH_B2B-XH-A_1x02_P2.50mm_Vertical, symbol Connector:Conn_01x02_Socket
- added J7: Conn_02x16_Odd_Even, Connector_PinHeader_2.54mm:PinHeader_2x16_P2.54mm_Vertical, symbol Connector_Generic:Conn_02x16_Odd_Even
Connections:
- net +3V3: now also J7.10 (Pin_10), J7.12 (Pin_12), J7.14 (Pin_14), J7.16 (Pin_16), J7.18 (Pin_18), J7.2 (Pin_2), J7.20 (Pin_20), J7.22 (Pin_22), J7.24 (Pin_24), J7.26 (Pin_26), J7.28 (Pin_28), J7.30 (Pin_30), J7.32 (Pin_32), J7.4 (Pin_4), J7.6 (Pin_6), J7.8 (Pin_8)
- net LIMIT1: now also J7.1 (Pin_1)
- net LIMIT10: now also J7.19 (Pin_19)
- net LIMIT11: now also J7.21 (Pin_21)
- net LIMIT12: now also J7.23 (Pin_23)
- net LIMIT13: now also J7.25 (Pin_25)
- net LIMIT14: now also J7.27 (Pin_27)
- net LIMIT16: now also J7.31 (Pin_31)
- net LIMIT2: now also J7.3 (Pin_3)
- net LIMIT3: now also J7.5 (Pin_5)
- net LIMIT4: now also J7.7 (Pin_7)
- net LIMIT5: now also J7.9 (Pin_9)
- net LIMIT6: now also J7.11 (Pin_11)
- net LIMIT8: now also J7.15 (Pin_15)
- net LIMIT9: now also J7.17 (Pin_17)
- net LIMIT_15 renamed LIMIT15
- net LIMIT15: now also J7.29 (Pin_29)
- net LIMIT_7 renamed LIMIT7
- net LIMIT7: now also J7.13 (Pin_13)

Commit message: メイン基板完成
Parts:
- renumbered R9 to R11, R10 to R12, R11 to R13, R12 to R14, R13 to R15, R14 to R16, R15 to R17, R16 to R18, R17 to R19, R18 to R20, R19 to R21, R20 to R22, R21 to R23, R22 to R24, R23 to R25, R24 to R26
