File: regulator.kicad_sch (KiCad schematic)
At the start: 37 parts, among them U1 XT30, U2 BP5293-50, U3 OKL-T/6-W12N-C, U4 BA033CC0FP

Commit message: 回路図だいたい完成
Parts:
- gave numbers to parts that had none: 15
Changed lines of the file:
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@@
 		(on_board yes)
 		(dnp no)
-		(property "Reference" "D?"
+		(property "Reference" "D7"
 			(at 142.24 39.37 0)
 			(effects
@@
 			(project "NHK2026_mainboard"
 				(path "/288b008e-4fe6-4fcf-a484-d519592de325/bbf41d6f-b9e1-40ca-b7d5-b0e7abfa8330"
-					(reference "D?")
+					(reference "D7")
 					(unit 1)
 				)
@@
 		(on_board yes)
 		(dnp no)
-		(property "Reference" "D?"
+		(property "Reference" "D11"
 			(at 245.11 60.96 90)
 			(effects
@@
 			(project "NHK2026_mainboard"
 				(path "/288b008e-4fe6-4fcf-a484-d519592de325/bbf41d6f-b9e1-40ca-b7d5-b0e7abfa8330"
-					(reference "D?")
+					(reference "D11")
 					(unit 1)
 				)
@@
 		(on_board yes)
 		(dnp no)
-		(property "Reference" "D?"
+		(property "Reference" "D6"
 			(at 115.57 49.53 0)
 			(effects
@@
 			(project "NHK2026_mainboard"
 				(path "/288b008e-4fe6-4fcf-a484-d519592de325/bbf41d6f-b9e1-40ca-b7d5-b0e7abfa8330"
-					(reference "D?")
+					(reference "D6")
 					(unit 1)
 				)
@@
 		(dnp no)
 		(fields_autoplaced yes)
-		(property "Reference" "RV?"
+		(property "Reference" "RV1"
 			(at 179.8321 107.3063 0)
 			(effects
@@
 			(project "NHK2026_mainboard"
 				(path "/288b008e-4fe6-4fcf-a484-d519592de325/bbf41d6f-b9e1-40ca-b7d5-b0e7abfa8330"
-					(reference "RV?")
+					(reference "RV1")
 					(unit 1)
 				)
@@
 		(dnp no)
 		(fields_autoplaced yes)
-		(property "Reference" "JP?"
+		(property "Reference" "JP1"
 			(at 144.653 114.9263 90)
 			(effects
@@
 			(project "NHK2026_mainboard"
 				(path "/288b008e-4fe6-4fcf-a484-d519592de325/bbf41d6f-b9e1-40ca-b7d5-b0e7abfa8330"
-					(reference "JP?")
+					(reference "JP1")
 					(unit 1)
 				)
@@
 		(dnp no)
 		(fields_autoplaced yes)
-		(property "Reference" "D?"
+		(property "Reference" "D1"
 			(at 67.31 133.0325 90)
 			(effects
@@
 			(project "NHK2026_mainboard"
 				(path "/288b008e-4fe6-4fcf-a484-d519592de325/bbf41d6f-b9e1-40ca-b7d5-b0e7abfa8330"
-					(reference "D?")
+					(reference "D1")
 					(unit 1)
 				)
@@
 		(dnp no)
 		(fields_autoplaced yes)
-		(property "Reference" "F?"
+		(property "Reference" "F1"
 			(at 100.33 48.26 90)
 			(effects
@@
 			(project "NHK2026_mainboard"
 				(path "/288b008e-4fe6-4fcf-a484-d519592de325/bbf41d6f-b9e1-40ca-b7d5-b0e7abfa8330"
-					(reference "F?")
+					(reference "F1")
 					(unit 1)
 				)
@@
 		(dnp no)
 		(fields_autoplaced yes)
-		(property "Reference" "D?"
+		(property "Reference" "D3"
 			(at 87.63 133.0325 90)
 			(effects
@@
 			(project "NHK2026_mainboard"
 				(path "/288b008e-4fe6-4fcf-a484-d519592de325/bbf41d6f-b9e1-40ca-b7d5-b0e7abfa8330"
-					(reference "D?")
+					(reference "D3")
 					(unit 1)
 				)
@@
 		(on_board yes)
 		(dnp no)
-		(property "Reference" "D?"
+		(property "Reference" "D8"
 			(at 166.37 60.96 90)
 			(effects
@@
 			(project "NHK2026_mainboard"
 				(path "/288b008e-4fe6-4fcf-a484-d519592de325/bbf41d6f-b9e1-40ca-b7d5-b0e7abfa8330"
-					(reference "D?")
+					(reference "D8")
 					(unit 1)
 				)
@@
 		(on_board yes)
 		(dnp no)
-		(property "Reference" "D?"
+		(property "Reference" "D5"
 			(at 109.22 108.585 90)
 			(effects
@@
 			(project "NHK2026_mainboard"
 				(path "/288b008e-4fe6-4fcf-a484-d519592de325/bbf41d6f-b9e1-40ca-b7d5-b0e7abfa8330"
-					(reference "D?")
+					(reference "D5")
 					(unit 1)
 				)
@@
 		(on_board yes)
 		(dnp no)
-		(property "Reference" "D?"
+		(property "Reference" "D9"
 			(at 205.74 39.37 0)
 			(effects
@@
 			(project "NHK2026_mainboard"
 				(path "/288b008e-4fe6-4fcf-a484-d519592de325/bbf41d6f-b9e1-40ca-b7d5-b0e7abfa8330"
-					(reference "D?")
+					(reference "D9")
 					(unit 1)
 				)
@@
 		(dnp no)
 		(fields_autoplaced yes)
-		(property "Reference" "D?"
+		(property "Reference" "D2"
 			(at 77.47 133.0325 90)
 			(effects
@@
 			(project "NHK2026_mainboard"
 				(path "/288b008e-4fe6-4fcf-a484-d519592de325/bbf41d6f-b9e1-40ca-b7d5-b0e7abfa8330"
-					(reference "D?")
+					(reference "D2")
 					(unit 1)
 				)
@@
 		(dnp no)
 		(fields_autoplaced yes)
-		(property "Reference" "D?"
+		(property "Reference" "D4"
 			(at 97.79 133.0325 90)
 			(effects
@@
 			(project "NHK2026_mainboard"
 				(path "/288b008e-4fe6-4fcf-a484-d519592de325/bbf41d6f-b9e1-40ca-b7d5-b0e7abfa8330"
-					(reference "D?")
+					(reference "D4")
 					(unit 1)
 				)
@@
 		(on_board yes)
 		(dnp no)
-		(property "Reference" "F?"
+		(property "Reference" "F2"
 			(at 100.33 90.17 90)
 			(effects
@@
 			(project "NHK2026_mainboard"
 				(path "/288b008e-4fe6-4fcf-a484-d519592de325/bbf41d6f-b9e1-40ca-b7d5-b0e7abfa8330"
-					(reference "F?")
+					(reference "F2")
 					(unit 1)
 				)
@@
 		(dnp no)
 		(fields_autoplaced yes)
-		(property "Reference" "D?"
+		(property "Reference" "D10"
 			(at 232.41 108.585 90)
 			(effects
@@
 			(project "NHK2026_mainboard"
 				(path "/288b008e-4fe6-4fcf-a484-d519592de325/bbf41d6f-b9e1-40ca-b7d5-b0e7abfa8330"
-					(reference "D?")
+					(reference "D10")
 					(unit 1)
 				)

Commit message: 何こっち見てんだよ
Parts:
- C9: renamed from C6; value 16v 100u -> 25v 470u; footprint Capacitor_THT:CP_Radial_D5.0mm_P2.00mm -> Capacitor_THT:CP_Radial_D8.0mm_P3.50mm
- D1, D2, D3, D4: footprint LED_THT:LED_D3.0mm -> LED_SMD:LED_0603_1608Metric_Pad1.05x0.95mm_HandSolder
- F1: value 0.5A 1A -> 0.65A 1.3A; footprint MyLib:PolyFuse_MF-NSMF-series -> Resistor_THT:R_Axial_DIN0207_L6.3mm_D2.5mm_P10.16mm_Horizontal
- U4: renamed from U1; footprint Connector_AMASS:AMASS_XT30U-M_1x02_P5.0mm_Vertical -> Connector_AMASS:AMASS_XT30PW-M_1x02_P2.50mm_Horizontal
- renumbered C7 to C10, C8 to C11, C9 to C12, C10 to C13, C11 to C14, C1 to C4, C2 to C5, C3 to C6, C4 to C7, C5 to C8, R1 to R2, R2 to R3, R3 to R4, R4 to R5, R5 to R6, R6 to R7, R7 to R8, U2 to U5, U3 to U6, U4 to U7

Commit message: 配線だいたい完了
Parts:
- F1: value 0.65A 1.3A -> MF-RX040; footprint Resistor_THT:R_Axial_DIN0207_L6.3mm_D2.5mm_P10.16mm_Horizontal -> Capacitor_THT:C_Disc_D10.0mm_W2.5mm_P5.00mm
Changed lines of the file:
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@@
 			)
 		)
-		(property "Value" "0.65A 1.3A"
+		(property "Value" "MF-RX040"
 			(at 100.33 50.8 90)
 			(effects
@@
 			)
 		)
-		(property "Footprint" "Resistor_THT:R_Axial_DIN0207_L6.3mm_D2.5mm_P10.16mm_Horizontal"
+		(property "Footprint" "Capacitor_THT:C_Disc_D10.0mm_W2.5mm_P5.00mm"
 			(at 105.41 53.34 0)
 			(effects

Commit message: メイン基板完成
Parts:
- renumbered D9 to D10, D10 to D11, D11 to D12, D1 to D2, D2 to D3, D3 to D4, D4 to D5, D5 to D6, D6 to D7, D7 to D8, D8 to D9, R8 to R10, R2 to R4, R3 to R5, R4 to R6, R5 to R7, R6 to R8, R7 to R9
