File: NHK2026_mainboard.kicad_pcb (KiCad board)
At the start: 2 copper layers, 100 x 100 mm, 151 parts, among them J1 ABS_Encoder, J10 LIMIT_13, J11 LIMIT_2, J12 LIMIT_6, J13 LIMIT_10, J14 LIMIT_14, J15 LIMIT_3, J16 LIMIT_7, J17 LIMIT_11, J18 LIMIT_15, J19 LIMIT_4, J2 SPI, J20 LIMIT_8, J21 LIMIT_12, J22 LIMIT_16, J23 RE_1, J24 RE_2, J25 RE_3, J26 RE_4, J27 RE_LPTIM1, J28 RE_LPTIM2, J29 RS485_1, J3 I2C, J30 RS485_2, J31 FDCAN_1, J32 FDCAN_2, J33 WTT12L_1, J34 WTT12L_2, J35 WTT12L_3, J36 DCMD1, J37 SERVO1, J38 DCMD2, J39 SERVO2, J4 SOLENOID_1, J40 DCMD3, J41 SERVO3, J42 DCMD4, J43 SERVO4, J5 ADC, J6 PicoScan, J7 LIMIT_1, J8 LIMIT_5, J9 LIMIT_9, SW1 SW_Push, U1 TXRX_pokayoke, U10 UTRS485G-S08-R, U11 UTRS485G-S08-R, U12 MCP2562-E-P, U13 MCP2562-E-P, U2 BNO055, U3 NUCLEO-H753ZI, U4 XT30, U5 BP5293-50, U6 OKL-T/6-W12N-C, U7 BA033CC0FP, U8 UTRS485G-S08-R, U9 UTRS485G-S08-R

Commit message: 配置だいたい完了
Parts:
- D6, D7, R39, R40, R41, R42, R43, R44, R45, R46, R47, R48, R49, R50, U10, U11, U8, U9: moved to B.Cu
- F1: value 0.65A 1.3A -> MF-RX040; footprint Resistor_THT:R_Axial_DIN0207_L6.3mm_D2.5mm_P10.16mm_Horizontal -> Capacitor_THT:C_Disc_D10.0mm_W2.5mm_P5.00mm
- moved J23 352.3 mm to (191.5, 128.3)
- moved U2 350.1 mm to (167.4, 137.2)
- moved J27 347.5 mm to (191.5, 138.4)
- moved J25 345.4 mm to (191.5, 108.5)
- moved J24 345.2 mm to (191.5, 98.6)
- moved J28 343.6 mm to (191.5, 118.4)
- moved U1 343.1 mm to (163.7, 148.5), turned to -90 degrees
- moved J26 342.6 mm to (191.5, 88.6)
- moved U12 322.8 mm to (183.9, 61.5)
- moved U13 313.0 mm to (183.9, 73.4)
- moved C3 306.2 mm to (130.5, 79.2), turned to 180 degrees
- moved D10 298.1 mm to (142.6, 112.8), turned to 180 degrees
- moved U6 290.7 mm to (145.0, 93.2), turned to -90 degrees
- moved C11 285.7 mm to (154.3, 99.9)
- moved C7 285.7 mm to (147.5, 83.3), turned to 180 degrees
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
Commit message: メイン基板完成
Parts:
- removed the J10 at (46.5, 145.3)
- removed the J11 at (55.9, 121.9)
- removed the J12 at (55.9, 129.7)
- removed the J13 at (55.9, 137.5)
- removed the J14 at (55.9, 145.3)
- removed the J15 at (65.4, 121.9)
- removed the J16 at (65.4, 129.7)
- removed the J17 at (65.4, 137.5)
- removed the J18 at (65.4, 145.3)
- removed the J19 at (74.8, 121.9)
- removed the J20 at (74.8, 129.7)
- removed the J21 at (74.8, 137.5)
- removed the J22 at (74.8, 145.3)
- removed the J8 at (46.5, 129.7)
- removed the J9 at (46.5, 137.5)
- added D1: LED, LED_SMD:LED_0603_1608Metric_Pad1.05x0.95mm_HandSolder, F.Cu at (111.1, 54.1)
- added R2: 1k, Resistor_SMD:R_0603_1608Metric_Pad0.98x0.95mm_HandSolder, F.Cu at (114.7, 54.1)
- added R3: 10k, Resistor_SMD:R_0603_1608Metric_Pad0.98x0.95mm_HandSolder, F.Cu at (109.6, 55.9)
- added SW2: SW_Push, Button_Switch_THT:SW_PUSH_6mm, F.Cu at (108.7, 58.2)
- added ref**: val**, MyLib:ROGIKEN, F.Cu at (189.2, 146.8)
- C15, C16, C17, C18, C19, C20, C21, C22, U1: moved to B.Cu
- D9: renamed from D8; moved to F.Cu
- J7: value LIMIT_1 -> Conn_02x16_Odd_Even; footprint Connector_JST:JST_XH_B2B-XH-A_1x02_P2.50mm_Vertical -> Connector_PinHeader_2.54mm:PinHeader_2x16_P2.54mm_Vertical
- R27: renamed from R25; moved to B.Cu
- R29: renamed from R27; moved to B.Cu
- R33: renamed from R31; moved to B.Cu
- R35: renamed from R33; moved to B.Cu
- R39: renamed from R37; moved to B.Cu
- R40: renamed from R38; moved to B.Cu
- RV1: value 20kB -> 140ohm
- U6: value OKL-T/6-W12N-C -> DCDC
- moved D4 335.8 mm to (172.8, 66.8), turned to 180 degrees
- moved D3 335.2 mm to (170.8, 54.4), turned to 180 degrees
- moved R14 308.4 mm to (158.5, 148.2), turned to 90 degrees
- moved R18 308.1 mm to (161.0, 148.2), turned to 90 degrees
- moved R5 307.9 mm to (167.3, 54.4)
- moved R22 307.7 mm to (163.6, 148.2), turned to 90 degrees
- moved R26 307.4 mm to (166.1, 148.2), turned to 90 degrees
- moved D5 306.2 mm to (148.8, 134.1)
- moved D6 306.0 mm to (150.2, 78.7)
- moved R6 301.1 mm to (169.3, 66.8)
- moved R13 299.4 mm to (148.3, 148.2), turned to 90 degrees
- moved R17 299.2 mm to (150.9, 148.2), turned to 90 degrees
- moved R21 298.6 mm to (153.4, 148.2), turned to 90 degrees
- moved R25 298.3 mm to (156.0, 148.2), turned to 90 degrees
- moved R12 290.5 mm to (138.2, 148.2), turned to 90 degrees
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- renumbered D9 to D10, D10 to D11, D11 to D12, D1 to D2, D2 to D3, D3 to D4, D4 to D5, D5 to D6, D6 to D7, D7 to D8, J25 to J10, J26 to J11, J27 to J12, J28 to J13, J29 to J14, J30 to J15, J31 to J16, J32 to J17, J33 to J18, J34 to J19, J35 to J20, J36 to J21, J37 to J22, J38 to J23, J39 to J24, J40 to J25, J41 to J26, J42 to J27, J43 to J28, J23 to J8, J24 to J9, R8 to R10, R9 to R11, R10 to R12, R11 to R13, R12 to R14, R13 to R15, R14 to R16, R15 to R17, R16 to R18, R17 to R19, R18 to R20, R19 to R21, R20 to R22, R21 to R23, R22 to R24, R23 to R25, R24 to R26, R26 to R28, R28 to R30, R29 to R31, R30 to R32, R32 to R34, R34 to R36, R35 to R37, R36 to R38, R2 to R4, R39 to R41, R40 to R42, R41 to R43, R42 to R44, R43 to R45, R44 to R46, R45 to R47, R46 to R48, R47 to R49, R3 to R5, R48 to R50, R49 to R51, R50 to R52, R4 to R6, R5 to R7, R6 to R8, R7 to R9
Connections:
- J5 pad 1: ADC_positive -> ADC_negative
- J5 pad 2: ADC_negative -> ADC_positive
- J7 pad 1: +3V3 -> LIMIT1
- J7 pad 2: LIMIT1 -> +3V3
- U3 pad CN11_1: unconnected-(U3A-PC10-PadCN11_1) -> USER_LED
- U3 pad CN11_9: unconnected-(U3A-PF6-PadCN11_9) -> USER_BUTTON
- U4 pad : (no net) -> GND
Routing:
- net GND: track 0.00 -> 1067.1 mm, vias 0 -> 634
- net +5V: track 0.00 -> 366.3 mm, vias 0 -> 10
- net +3V3: track 0.00 -> 328.5 mm
- net LIMIT12: track 0.00 -> 127.0 mm, vias 0 -> 1
- net RS485_1TX: track 0.00 -> 113.6 mm, vias 0 -> 1
- net RS485_1RX: track 0.00 -> 102.8 mm, vias 0 -> 1
- net +5VP: track 0.00 -> 98.2 mm
- net +12V: track 0.00 -> 95.8 mm, vias 0 -> 1
- net ENC_LPTIM_1B: track 0.00 -> 90.6 mm
- net WTT12L_1Q2: track 0.00 -> 85.9 mm, vias 0 -> 2
- net ENC_2A: track 0.00 -> 85.7 mm
- net ENC_LPTIM_1A: track 0.00 -> 78.6 mm
- net WTT12L_3Q2: track 0.00 -> 65.6 mm
- net WTT12L_2Q2: track 0.00 -> 65.1 mm
- net LIMIT13: track 0.00 -> 63.2 mm
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- added copper zone on B.Cu, net GND
- added copper zone on F.Cu, net GND
Other:
- board text added: "->RX:A"
- board text added: "->RX:B"
- board text added: "12V"
- board text added: "12v"
- board text added: "3V3"
- board text added: "5V"
- board text added: "5VP"
- board text added: "<-TX:A"
- board text added: "<-TX:B"
- board text added: "ABS_ENC"
- board text added: "ADC"
- board text added: "ADC_1"
- board text added: "BNO"
- board text added: "CAN"
- board text added: "CAN_H"
- board text added: "CAN_L"
- board text added: "CH1"
- board text added: "CH1↑"
- board text added: "CH2"
- board text added: "CH2↑"
- board text added: "CH3"
- board text added: "CH4"
- board text added: "CS"
- board text added: "DCMD_TIM3"
- board text added: "DIR"
- board text added: "FDCAN_1"
- board text added: "FDCAN_2"
- board text added: "GND"
- board text added: "I2C"
- board text added: "INC_ENC"
- board text added: "Ilias2026_mainboard Rev1.0 @KayOChef_meme"
- board text added: "LIMIT_SW"
- board text added: "LPTIM1"
- board text added: "LPTIM2"
- board text added: "LiDAR"
- board text added: "MISO"
- board text added: "MOSI"
- board text added: "N"
- board text added: "PA13"
- board text added: "PA14"
- board text added: "PA15"
- board text added: "PA4"
- board text added: "PB11"
- board text added: "PC11"
- board text added: "PC12"
- board text added: "PE10"
- board text added: "PE12"
- board text added: "PE13"
- board text added: "PE14"
- board text added: "PE15"
- board text added: "PF13"
- board text added: "PF14"
- board text added: "PF15"
- board text added: "PF9"
- board text added: "PG0"
- board text added: "PG1"
- board text added: "PG10"
- board text added: "PG2"
- board text added: "PG3"
- board text added: "PG4"
- board text added: "PG5"
- board text added: "PG6"
- board text added: "PG7"
- board text added: "PG8"
- board text added: "PWM"
- board text added: "RESET"
- board text added: "RS-485"
- board text added: "SCK"
- board text added: "SERVO"
- board text added: "SOLENOID"
- board text added: "SPI"
- board text added: "SPI2"
- board text added: "SPI_1"
- board text added: "TIM1"
- board text added: "TIM12"
- board text added: "TIM15"
- board text added: "TIM2"
- board text added: "TIM4"
- board text added: "TIM8"
- board text added: "USART1"
- board text added: "USART2"
- board text added: "USART6"
- board text added: "USER PC10"
- board text added: "USER PF6"
- board text added: "WTT12L"
- board text added: "p"
- board text added: "↓CH1"
- board text added: "↓CH2"
- board text added: "↓PF10"
- board text added: "↓PF3"
- board text added: "↓PF4"
- board text added: "↓PF5"

Commit message: QRコードと回路図pdfを追加
Parts:
- added G***: LOGO, QRcode:Ilias2026_mainboard, B.Cu at (184.7, 54.6)

Commit message: 製造番号位置指定
Other:
- board text added: "JLCJLCJLCJLC"
Changed lines of the file:
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@@
+		)
+	)
+	(gr_text "JLCJLCJLCJLC"
+		(at 186.944 87.376 0)
+		(layer "F.SilkS")
+		(effects
+			(font
+				(size 1 1)
+				(thickness 0.1)
+			)
+			(justify left bottom)
 		)
 	)

Commit message: 微修正
Parts:
- added C15: 0.1u, Capacitor_SMD:C_0603_1608Metric_Pad1.08x0.95mm_HandSolder, B.Cu at (193.2, 125.7)
- added C16: 0.1u, Capacitor_SMD:C_0603_1608Metric_Pad1.08x0.95mm_HandSolder, B.Cu at (193.2, 96.5)
- added C17: 0.1u, Capacitor_SMD:C_0603_1608Metric_Pad1.08x0.95mm_HandSolder, B.Cu at (193.2, 106.4)
- added C18: 0.1u, Capacitor_SMD:C_0603_1608Metric_Pad1.08x0.95mm_HandSolder, B.Cu at (193.6, 86.1)
- added C19: 0.1u, Capacitor_SMD:C_0603_1608Metric_Pad1.08x0.95mm_HandSolder, B.Cu at (193.2, 136.4)
- added C20: 0.1u, Capacitor_SMD:C_0603_1608Metric_Pad1.08x0.95mm_HandSolder, B.Cu at (193.2, 116.3)
- added C30: 25V 470u, Capacitor_THT:CP_Radial_D8.0mm_P3.50mm, F.Cu at (129.8, 81.9)
- added C33: 0.1u, Capacitor_SMD:C_0603_1608Metric_Pad1.08x0.95mm_HandSolder, B.Cu at (142.5, 122.9)
- added C34: 0.1u, Capacitor_SMD:C_0603_1608Metric_Pad1.08x0.95mm_HandSolder, B.Cu at (142.6, 127.0)
- added C35: 0.1u, Capacitor_SMD:C_0603_1608Metric_Pad1.08x0.95mm_HandSolder, B.Cu at (151.8, 125.7)
- added C36: 0.1u, Capacitor_SMD:C_0603_1608Metric_Pad1.08x0.95mm_HandSolder, B.Cu at (151.9, 121.9)
- RV1: value 140ohm -> 20kB
- U6: value DCDC -> OKL-T/6-W12N-C
- moved J6 9.14 mm to (129.8, 74.7)
- moved C3 8.89 mm to (128.9, 69.8)
- moved C1 2.84 mm to (167.1, 126.3)
- renumbered C15 to C21, C16 to C22, C17 to C23, C18 to C24, C19 to C25, C20 to C26, C21 to C27, C22 to C28, C23 to C29, C24 to C31, C25 to C32
Routing:
- net +5V: track 366.3 -> 377.0 mm
- net GND: track 1067.1 -> 1077.1 mm, vias 634 -> 627
- net +5VP: track 98.2 -> 107.3 mm
- net ENC_LPTIM_1B: track 90.6 -> 93.5 mm
- net ENC_LPTIM_2B: track 22.8 -> 24.3 mm
- net ENC_2B: track 23.0 -> 24.1 mm
- net ENC_3B: track 21.9 -> 22.7 mm
