File: encoder.kicad_sch (KiCad schematic)
At the start: 6 parts, among them J1 RE_3, J2 RE_4, J3 RE_LPTIM1, J4 RE_LPTIM2

Commit message: 回路図だいたい完成
Parts:
- gave numbers to parts that had none: 2
Changed lines of the file:
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@@
 		(dnp no)
 		(fields_autoplaced yes)
-		(property "Reference" "#PWR?"
+		(property "Reference" "#PWR0147"
 			(at 36.83 31.75 0)
 			(effects
@@
 			(project "NHK2026_mainboard"
 				(path "/288b008e-4fe6-4fcf-a484-d519592de325/a2277374-1148-40a7-b5a9-92fb07a5018d"
-					(reference "#PWR?")
+					(reference "#PWR0147")
 					(unit 1)
 				)
@@
 		(dnp no)
 		(fields_autoplaced yes)
-		(property "Reference" "#PWR?"
+		(property "Reference" "#PWR0146"
 			(at 71.12 49.53 0)
 			(effects
@@
 			(project "NHK2026_mainboard"
 				(path "/288b008e-4fe6-4fcf-a484-d519592de325/a2277374-1148-40a7-b5a9-92fb07a5018d"
-					(reference "#PWR?")
+					(reference "#PWR0146")
 					(unit 1)
 				)
@@
 		(dnp no)
 		(fields_autoplaced yes)
-		(property "Reference" "#PWR?"
+		(property "Reference" "#PWR0145"
 			(at 69.85 31.75 0)
 			(effects
@@
 			(project "NHK2026_mainboard"
 				(path "/288b008e-4fe6-4fcf-a484-d519592de325/a2277374-1148-40a7-b5a9-92fb07a5018d"
-					(reference "#PWR?")
+					(reference "#PWR0145")
 					(unit 1)
 				)
@@
 		(dnp no)
 		(fields_autoplaced yes)
-		(property "Reference" "#PWR?"
+		(property "Reference" "#PWR0148"
 			(at 38.1 49.53 0)
 			(effects
@@
 			(project "NHK2026_mainboard"
 				(path "/288b008e-4fe6-4fcf-a484-d519592de325/a2277374-1148-40a7-b5a9-92fb07a5018d"
-					(reference "#PWR?")
+					(reference "#PWR0148")
 					(unit 1)
 				)
@@
 		(on_board yes)
 		(dnp no)
-		(property "Reference" "J?"
+		(property "Reference" "J34"
 			(at 48.895 34.909 0)
 			(effects
@@
 			(project "NHK2026_mainboard"
 				(path "/288b008e-4fe6-4fcf-a484-d519592de325/a2277374-1148-40a7-b5a9-92fb07a5018d"
-					(reference "J?")
+					(reference "J34")
 					(unit 1)
 				)
@@
 		(on_board yes)
 		(dnp no)
-		(property "Reference" "J?"
+		(property "Reference" "J35"
 			(at 81.915 34.909 0)
 			(effects
@@
 			(project "NHK2026_mainboard"
 				(path "/288b008e-4fe6-4fcf-a484-d519592de325/a2277374-1148-40a7-b5a9-92fb07a5018d"
-					(reference "J?")
-					(unit 1)
-				)
+					(reference "J35")
+					(unit 1)
+				)

Commit message: 何こっち見てんだよ
Parts:
- renumbered J34 to J23, J35 to J24, J1 to J25, J2 to J26, J3 to J27, J4 to J28

Commit message: 配線だいたい完了
Parts:
- renumbered J25 to J10, J26 to J11, J27 to J12, J28 to J13, J23 to J8, J24 to J9
Changed lines of the file:
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@@
 		(dnp no)
 		(fields_autoplaced yes)
-		(property "Reference" "#PWR075"
+		(property "Reference" "#PWR060"
 			(at 101.6 31.75 0)
 			(effects
@@
 			(project "NHK2026_mainboard"
 				(path "/288b008e-4fe6-4fcf-a484-d519592de325/a2277374-1148-40a7-b5a9-92fb07a5018d"
-					(reference "#PWR075")
+					(reference "#PWR060")
 					(unit 1)
 				)
@@
 		(dnp no)
 		(fields_autoplaced yes)
-		(property "Reference" "#PWR076"
+		(property "Reference" "#PWR061"
 			(at 102.87 49.53 0)
 			(effects
@@
 			(project "NHK2026_mainboard"
 				(path "/288b008e-4fe6-4fcf-a484-d519592de325/a2277374-1148-40a7-b5a9-92fb07a5018d"
-					(reference "#PWR076")
+					(reference "#PWR061")
 					(unit 1)
 				)
@@
 		(dnp no)
 		(fields_autoplaced yes)
-		(property "Reference" "#PWR079"
+		(property "Reference" "#PWR064"
 			(at 170.18 31.75 0)
 			(effects
@@
 			(project "NHK2026_mainboard"
 				(path "/288b008e-4fe6-4fcf-a484-d519592de325/a2277374-1148-40a7-b5a9-92fb07a5018d"
-					(reference "#PWR079")
+					(reference "#PWR064")
 					(unit 1)
 				)
@@
 		(dnp no)
 		(fields_autoplaced yes)
-		(property "Reference" "#PWR071"
+		(property "Reference" "#PWR056"
 			(at 36.83 31.75 0)
 			(effects
@@
 			(project "NHK2026_mainboard"
 				(path "/288b008e-4fe6-4fcf-a484-d519592de325/a2277374-1148-40a7-b5a9-92fb07a5018d"
-					(reference "#PWR071")
+					(reference "#PWR056")
 					(unit 1)
 				)
@@
 		(dnp no)
 		(fields_autoplaced yes)
-		(property "Reference" "#PWR074"
+		(property "Reference" "#PWR059"
 			(at 71.12 49.53 0)
 			(effects
@@
 			(project "NHK2026_mainboard"
 				(path "/288b008e-4fe6-4fcf-a484-d519592de325/a2277374-1148-40a7-b5a9-92fb07a5018d"
-					(reference "#PWR074")
+					(reference "#PWR059")
 					(unit 1)
 				)
@@
 		(on_board yes)
 		(dnp no)
-		(property "Reference" "J25"
+		(property "Reference" "J10"
 			(at 113.665 34.909 0)
 			(effects
@@
 			(project "NHK2026_mainboard"
 				(path "/288b008e-4fe6-4fcf-a484-d519592de325/a2277374-1148-40a7-b5a9-92fb07a5018d"
-					(reference "J25")
+					(reference "J10")
 					(unit 1)
 				)
@@
 		(dnp no)
 		(fields_autoplaced yes)
-		(property "Reference" "#PWR082"
+		(property "Reference" "#PWR067"
 			(at 212.09 49.53 0)
 			(effects
@@
 			(project "NHK2026_mainboard"
 				(path "/288b008e-4fe6-4fcf-a484-d519592de325/a2277374-1148-40a7-b5a9-92fb07a5018d"
-					(reference "#PWR082")
+					(reference "#PWR067")
 					(unit 1)
 				)
@@
 		(dnp no)
 		(fields_autoplaced yes)
-		(property "Reference" "#PWR078"
+		(property "Reference" "#PWR063"
 			(at 134.62 49.53 0)
 			(effects
@@
 			(project "NHK2026_mainboard"
 				(path "/288b008e-4fe6-4fcf-a484-d519592de325/a2277374-1148-40a7-b5a9-92fb07a5018d"
-					(reference "#PWR078")
+					(reference "#PWR063")
 					(unit 1)
 				)
@@
 		(dnp no)
 		(fields_autoplaced yes)
-		(property "Reference" "#PWR081"
+		(property "Reference" "#PWR066"
 			(at 210.82 31.75 0)
 			(effects
@@
 			(project "NHK2026_mainboard"
 				(path "/288b008e-4fe6-4fcf-a484-d519592de325/a2277374-1148-40a7-b5a9-92fb07a5018d"
-					(reference "#PWR081")
+					(reference "#PWR066")
 					(unit 1)
 				)
@@
 		(dnp no)
 		(fields_autoplaced yes)
-		(property "Reference" "#PWR080"
+		(property "Reference" "#PWR065"
 			(at 171.45 49.53 0)
 			(effects
@@
 			(project "NHK2026_mainboard"
 				(path "/288b008e-4fe6-4fcf-a484-d519592de325/a2277374-1148-40a7-b5a9-92fb07a5018d"
-					(reference "#PWR080")
+					(reference "#PWR065")
 					(unit 1)
 				)
@@
 		(dnp no)
 		(fields_autoplaced yes)
-		(property "Reference" "#PWR077"
+		(property "Reference" "#PWR062"
 			(at 133.35 31.75 0)
 			(effects
@@
 			(project "NHK2026_mainboard"
 				(path "/288b008e-4fe6-4fcf-a484-d519592de325/a2277374-1148-40a7-b5a9-92fb07a5018d"
-					(reference "#PWR077")
+					(reference "#PWR062")
 					(unit 1)
 				)
@@
 		(dnp no)
 		(fields_autoplaced yes)
-		(property "Reference" "#PWR073"
+		(property "Reference" "#PWR058"
 			(at 69.85 31.75 0)
 			(effects
@@
 			(project "NHK2026_mainboard"
 				(path "/288b008e-4fe6-4fcf-a484-d519592de325/a2277374-1148-40a7-b5a9-92fb07a5018d"
-					(reference "#PWR073")
+					(reference "#PWR058")
 					(unit 1)
 				)
@@
 		(on_board yes)
 		(dnp no)
-		(property "Reference" "J26"
+		(property "Reference" "J11"
 			(at 145.415 34.909 0)
 			(effects
@@
 			(project "NHK2026_mainboard"
 				(path "/288b008e-4fe6-4fcf-a484-d519592de325/a2277374-1148-40a7-b5a9-92fb07a5018d"
-					(reference "J26")
+					(reference "J11")
 					(unit 1)
 				)
@@
 		(dnp no)
 		(fields_autoplaced yes)
-		(property "Reference" "#PWR072"
+		(property "Reference" "#PWR057"
 			(at 38.1 49.53 0)
 			(effects
@@
 			(project "NHK2026_mainboard"
 				(path "/288b008e-4fe6-4fcf-a484-d519592de325/a2277374-1148-40a7-b5a9-92fb07a5018d"
-					(reference "#PWR072")
+					(reference "#PWR057")
 					(unit 1)
 				)
@@
 		(on_board yes)
 		(dnp no)
-		(property "Reference" "J23"
+		(property "Reference" "J8"
 			(at 48.895 34.909 0)
 			(effects
@@
 			(project "NHK2026_mainboard"
 				(path "/288b008e-4fe6-4fcf-a484-d519592de325/a2277374-1148-40a7-b5a9-92fb07a5018d"
-					(reference "J23")
+					(reference "J8")
 					(unit 1)
 				)
@@
 		(on_board yes)
 		(dnp no)
-		(property "Reference" "J28"
+		(property "Reference" "J13"
 			(at 222.885 34.909 0)
 			(effects
@@
 			(project "NHK2026_mainboard"
 				(path "/288b008e-4fe6-4fcf-a484-d519592de325/a2277374-1148-40a7-b5a9-92fb07a5018d"
-					(reference "J28")
+					(reference "J13")
 					(unit 1)
 				)
@@
 		(on_board yes)
 		(dnp no)
-		(property "Reference" "J24"
+		(property "Reference" "J9"
 			(at 81.915 34.909 0)
 			(effects
@@
 			(project "NHK2026_mainboard"
 				(path "/288b008e-4fe6-4fcf-a484-d519592de325/a2277374-1148-40a7-b5a9-92fb07a5018d"
-					(reference "J24")
+					(reference "J9")
 					(unit 1)
 				)
@@
 		(on_board yes)
 		(dnp no)
-		(property "Reference" "J27"
+		(property "Reference" "J12"
 			(at 182.245 34.909 0)
 			(effects
@@
 			(project "NHK2026_mainboard"
 				(path "/288b008e-4fe6-4fcf-a484-d519592de325/a2277374-1148-40a7-b5a9-92fb07a5018d"
-					(reference "J27")
-					(unit 1)
-				)
+					(reference "J12")
+					(unit 1)
+				)

Commit message: 微修正
Parts:
- added C15, C16, C17, C18, C19, C20: 0.1u, Capacitor_SMD:C_0603_1608Metric_Pad1.08x0.95mm_HandSolder, symbol Device:C
Connections:
- net +5V: now also C15.1, C16.1, C17.1, C18.1, C19.1, C20.1
- net GND: now also C15.2, C16.2, C17.2, C18.2, C19.2, C20.2
