File: motor.kicad_sch (KiCad schematic)
At the start: 8 parts, among them J10 SERVO3, J11 DCMD4, J12 SERVO4, J5 DCMD1, J6 SERVO1, J7 DCMD2, J8 SERVO2, J9 DCMD3

Commit message: 何こっち見てんだよ
Parts:
- J36: renamed from J5; footprint (none) -> Connector_JST:JST_XH_B3B-XH-A_1x03_P2.50mm_Vertical
- J37: renamed from J6; footprint (none) -> Connector_JST:JST_XH_B3B-XH-A_1x03_P2.50mm_Vertical
- J38: renamed from J7; footprint (none) -> Connector_JST:JST_XH_B3B-XH-A_1x03_P2.50mm_Vertical
- J39: renamed from J8; footprint (none) -> Connector_JST:JST_XH_B3B-XH-A_1x03_P2.50mm_Vertical
- J40: renamed from J9; footprint (none) -> Connector_JST:JST_XH_B3B-XH-A_1x03_P2.50mm_Vertical
- J41: renamed from J10; footprint (none) -> Connector_JST:JST_XH_B3B-XH-A_1x03_P2.50mm_Vertical
- J42: renamed from J11; footprint (none) -> Connector_JST:JST_XH_B3B-XH-A_1x03_P2.50mm_Vertical
- J43: renamed from J12; footprint (none) -> Connector_JST:JST_XH_B3B-XH-A_1x03_P2.50mm_Vertical
Other:
- note added: "DCMD"
- note added: "SERVO"

Commit message: 配線だいたい完了
Parts:
- renumbered J36 to J21, J37 to J22, J38 to J23, J39 to J24, J40 to J25, J41 to J26, J42 to J27, J43 to J28
Changed lines of the file:
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@@
 		(on_board yes)
 		(dnp no)
-		(property "Reference" "J36"
+		(property "Reference" "J21"
 			(at 68.58 72.3901 0)
 			(effects
@@
 			(project "NHK2026_mainboard"
 				(path "/288b008e-4fe6-4fcf-a484-d519592de325/4c5acf8a-e8b2-46e6-aff7-72cd28b0a4c6"
-					(reference "J36")
+					(reference "J21")
 					(unit 1)
 				)
@@
 		(dnp no)
 		(fields_autoplaced yes)
-		(property "Reference" "#PWR0144"
+		(property "Reference" "#PWR0129"
 			(at 144.78 121.92 0)
 			(effects
@@
 			(project "NHK2026_mainboard"
 				(path "/288b008e-4fe6-4fcf-a484-d519592de325/4c5acf8a-e8b2-46e6-aff7-72cd28b0a4c6"
-					(reference "#PWR0144")
+					(reference "#PWR0129")
 					(unit 1)
 				)
@@
 		(dnp no)
 		(fields_autoplaced yes)
-		(property "Reference" "#PWR0142"
+		(property "Reference" "#PWR0127"
 			(at 144.78 83.82 0)
 			(effects
@@
 			(project "NHK2026_mainboard"
 				(path "/288b008e-4fe6-4fcf-a484-d519592de325/4c5acf8a-e8b2-46e6-aff7-72cd28b0a4c6"
-					(reference "#PWR0142")
+					(reference "#PWR0127")
 					(unit 1)
 				)
@@
 		(on_board yes)
 		(dnp no)
-		(property "Reference" "J40"
+		(property "Reference" "J25"
 			(at 124.46 72.3901 0)
 			(effects
@@
 			(project "NHK2026_mainboard"
 				(path "/288b008e-4fe6-4fcf-a484-d519592de325/4c5acf8a-e8b2-46e6-aff7-72cd28b0a4c6"
-					(reference "J40")
+					(reference "J25")
 					(unit 1)
 				)
@@
 		(on_board yes)
 		(dnp no)
-		(property "Reference" "J43"
+		(property "Reference" "J28"
 			(at 152.4 110.4901 0)
 			(effects
@@
 			(project "NHK2026_mainboard"
 				(path "/288b008e-4fe6-4fcf-a484-d519592de325/4c5acf8a-e8b2-46e6-aff7-72cd28b0a4c6"
-					(reference "J43")
+					(reference "J28")
 					(unit 1)
 				)
@@
 		(dnp no)
 		(fields_autoplaced yes)
-		(property "Reference" "#PWR0137"
+		(property "Reference" "#PWR0122"
 			(at 88.9 107.95 0)
 			(effects
@@
 			(project "NHK2026_mainboard"
 				(path "/288b008e-4fe6-4fcf-a484-d519592de325/4c5acf8a-e8b2-46e6-aff7-72cd28b0a4c6"
-					(reference "#PWR0137")
+					(reference "#PWR0122")
 					(unit 1)
 				)
@@
 		(dnp no)
 		(fields_autoplaced yes)
-		(property "Reference" "#PWR0141"
+		(property "Reference" "#PWR0126"
 			(at 116.84 121.92 0)
 			(effects
@@
 			(project "NHK2026_mainboard"
 				(path "/288b008e-4fe6-4fcf-a484-d519592de325/4c5acf8a-e8b2-46e6-aff7-72cd28b0a4c6"
-					(reference "#PWR0141")
+					(reference "#PWR0126")
 					(unit 1)
 				)
@@
 		(on_board yes)
 		(dnp no)
-		(property "Reference" "J37"
+		(property "Reference" "J22"
 			(at 68.58 110.4901 0)
 			(effects
@@
 			(project "NHK2026_mainboard"
 				(path "/288b008e-4fe6-4fcf-a484-d519592de325/4c5acf8a-e8b2-46e6-aff7-72cd28b0a4c6"
-					(reference "J37")
+					(reference "J22")
 					(unit 1)
 				)
@@
 		(dnp no)
 		(fields_autoplaced yes)
-		(property "Reference" "#PWR0139"
+		(property "Reference" "#PWR0124"
 			(at 116.84 83.82 0)
 			(effects
@@
 			(project "NHK2026_mainboard"
 				(path "/288b008e-4fe6-4fcf-a484-d519592de325/4c5acf8a-e8b2-46e6-aff7-72cd28b0a4c6"
-					(reference "#PWR0139")
+					(reference "#PWR0124")
 					(unit 1)
 				)
@@
 		(dnp no)
 		(fields_autoplaced yes)
-		(property "Reference" "#PWR0136"
+		(property "Reference" "#PWR0121"
 			(at 88.9 83.82 0)
 			(effects
@@
 			(project "NHK2026_mainboard"
 				(path "/288b008e-4fe6-4fcf-a484-d519592de325/4c5acf8a-e8b2-46e6-aff7-72cd28b0a4c6"
-					(reference "#PWR0136")
+					(reference "#PWR0121")
 					(unit 1)
 				)
@@
 		(on_board yes)
 		(dnp no)
-		(property "Reference" "J41"
+		(property "Reference" "J26"
 			(at 124.46 110.4901 0)
 			(effects
@@
 			(project "NHK2026_mainboard"
 				(path "/288b008e-4fe6-4fcf-a484-d519592de325/4c5acf8a-e8b2-46e6-aff7-72cd28b0a4c6"
-					(reference "J41")
+					(reference "J26")
 					(unit 1)
 				)
@@
 		(on_board yes)
 		(dnp no)
-		(property "Reference" "J38"
+		(property "Reference" "J23"
 			(at 96.52 72.3901 0)
 			(effects
@@
 			(project "NHK2026_mainboard"
 				(path "/288b008e-4fe6-4fcf-a484-d519592de325/4c5acf8a-e8b2-46e6-aff7-72cd28b0a4c6"
-					(reference "J38")
+					(reference "J23")
 					(unit 1)
 				)
@@
 		(on_board yes)
 		(dnp no)
-		(property "Reference" "J42"
+		(property "Reference" "J27"
 			(at 152.4 72.3901 0)
 			(effects
@@
 			(project "NHK2026_mainboard"
 				(path "/288b008e-4fe6-4fcf-a484-d519592de325/4c5acf8a-e8b2-46e6-aff7-72cd28b0a4c6"
-					(reference "J42")
+					(reference "J27")
 					(unit 1)
 				)
@@
 		(dnp no)
 		(fields_autoplaced yes)
-		(property "Reference" "#PWR0143"
+		(property "Reference" "#PWR0128"
 			(at 144.78 107.95 0)
 			(effects
@@
 			(project "NHK2026_mainboard"
 				(path "/288b008e-4fe6-4fcf-a484-d519592de325/4c5acf8a-e8b2-46e6-aff7-72cd28b0a4c6"
-					(reference "#PWR0143")
+					(reference "#PWR0128")
 					(unit 1)
 				)
@@
 		(dnp no)
 		(fields_autoplaced yes)
-		(property "Reference" "#PWR0134"
+		(property "Reference" "#PWR0119"
 			(at 60.96 107.95 0)
 			(effects
@@
 			(project "NHK2026_mainboard"
 				(path "/288b008e-4fe6-4fcf-a484-d519592de325/4c5acf8a-e8b2-46e6-aff7-72cd28b0a4c6"
-					(reference "#PWR0134")
+					(reference "#PWR0119")
 					(unit 1)
 				)
@@
 		(dnp no)
 		(fields_autoplaced yes)
-		(property "Reference" "#PWR0135"
+		(property "Reference" "#PWR0120"
 			(at 60.96 121.92 0)
 			(effects
@@
 			(project "NHK2026_mainboard"
 				(path "/288b008e-4fe6-4fcf-a484-d519592de325/4c5acf8a-e8b2-46e6-aff7-72cd28b0a4c6"
-					(reference "#PWR0135")
+					(reference "#PWR0120")
 					(unit 1)
 				)
@@
 		(on_board yes)
 		(dnp no)
-		(property "Reference" "J39"
+		(property "Reference" "J24"
 			(at 96.52 110.4901 0)
 			(effects
@@
 			(project "NHK2026_mainboard"
 				(path "/288b008e-4fe6-4fcf-a484-d519592de325/4c5acf8a-e8b2-46e6-aff7-72cd28b0a4c6"
-					(reference "J39")
+					(reference "J24")
 					(unit 1)
 				)
@@
 		(dnp no)
 		(fields_autoplaced yes)
-		(property "Reference" "#PWR0138"
+		(property "Reference" "#PWR0123"
 			(at 88.9 121.92 0)
 			(effects
@@
 			(project "NHK2026_mainboard"
 				(path "/288b008e-4fe6-4fcf-a484-d519592de325/4c5acf8a-e8b2-46e6-aff7-72cd28b0a4c6"
-					(reference "#PWR0138")
+					(reference "#PWR0123")
 					(unit 1)
 				)
@@
 		(dnp no)
 		(fields_autoplaced yes)
-		(property "Reference" "#PWR0133"
+		(property "Reference" "#PWR0118"
 			(at 60.96 83.82 0)
 			(effects
@@
 			(project "NHK2026_mainboard"
 				(path "/288b008e-4fe6-4fcf-a484-d519592de325/4c5acf8a-e8b2-46e6-aff7-72cd28b0a4c6"
-					(reference "#PWR0133")
+					(reference "#PWR0118")
 					(unit 1)
 				)
@@
 		(dnp no)
 		(fields_autoplaced yes)
-		(property "Reference" "#PWR0140"
+		(property "Reference" "#PWR0125"
 			(at 116.84 107.95 0)
 			(effects
@@
 			(project "NHK2026_mainboard"
 				(path "/288b008e-4fe6-4fcf-a484-d519592de325/4c5acf8a-e8b2-46e6-aff7-72cd28b0a4c6"
-					(reference "#PWR0140")
-					(unit 1)
-				)
+					(reference "#PWR0125")
+					(unit 1)
+				)

Commit message: 微修正
Parts:
- added C33, C34, C35, C36: 0.1u, Capacitor_SMD:C_0603_1608Metric_Pad1.08x0.95mm_HandSolder, symbol Device:C
Connections:
- net +5VP: now also C33.1, C34.1, C35.1, C36.1
- net GND: now also C33.2, C34.2, C35.2, C36.2
