File: rs485.kicad_sch (KiCad schematic)
At the start: 22 parts

Commit message: 回路図だいたい完成
Parts:
- gave numbers to parts that had none: 22

Commit message: 何こっち見てんだよ
Parts:
- J29: renamed from J36; footprint Connector_JST:JST_XH_S5B-XH-A-1_1x05_P2.50mm_Horizontal -> Connector_JST:JST_XH_B5B-XH-A_1x05_P2.50mm_Vertical
- J30: renamed from J37; value RS485_1 -> RS485_2; footprint Connector_JST:JST_XH_S5B-XH-A-1_1x05_P2.50mm_Horizontal -> Connector_JST:JST_XH_B5B-XH-A_1x05_P2.50mm_Vertical
- renumbered C14 to C15, C15 to C16, C16 to C17, C17 to C18, R24 to R25, R25 to R26, R26 to R27, R27 to R28, R28 to R29, R29 to R30, R30 to R31, R31 to R32, R32 to R33, R33 to R34, R34 to R35, R35 to R36

Commit message: 配線だいたい完了
Parts:
- renumbered J29 to J14, J30 to J15
Changed lines of the file:
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@@
 		(dnp no)
 		(fields_autoplaced yes)
-		(property "Reference" "#PWR088"
+		(property "Reference" "#PWR073"
 			(at 67.945 88.9 0)
 			(effects
@@
 			(project "NHK2026_mainboard"
 				(path "/288b008e-4fe6-4fcf-a484-d519592de325/6ae9977e-919b-4292-b0e6-ff735491d0d2"
-					(reference "#PWR088")
+					(reference "#PWR073")
 					(unit 1)
 				)
@@
 		(dnp no)
 		(fields_autoplaced yes)
-		(property "Reference" "#PWR096"
+		(property "Reference" "#PWR081"
 			(at 179.705 49.53 0)
 			(effects
@@
 			(project "NHK2026_mainboard"
 				(path "/288b008e-4fe6-4fcf-a484-d519592de325/6ae9977e-919b-4292-b0e6-ff735491d0d2"
-					(reference "#PWR096")
+					(reference "#PWR081")
 					(unit 1)
 				)
@@
 		(dnp no)
 		(fields_autoplaced yes)
-		(property "Reference" "#PWR086"
+		(property "Reference" "#PWR071"
 			(at 46.355 68.58 0)
 			(effects
@@
 			(project "NHK2026_mainboard"
 				(path "/288b008e-4fe6-4fcf-a484-d519592de325/6ae9977e-919b-4292-b0e6-ff735491d0d2"
-					(reference "#PWR086")
+					(reference "#PWR071")
 					(unit 1)
 				)
@@
 		(dnp no)
 		(fields_autoplaced yes)
-		(property "Reference" "J30"
+		(property "Reference" "J15"
 			(at 222.25 86.3599 0)
 			(effects
@@
 			(project "NHK2026_mainboard"
 				(path "/288b008e-4fe6-4fcf-a484-d519592de325/6ae9977e-919b-4292-b0e6-ff735491d0d2"
-					(reference "J30")
+					(reference "J15")
 					(unit 1)
 				)
@@
 		(dnp no)
 		(fields_autoplaced yes)
-		(property "Reference" "#PWR092"
+		(property "Reference" "#PWR077"
 			(at 156.845 121.92 0)
 			(effects
@@
 			(project "NHK2026_mainboard"
 				(path "/288b008e-4fe6-4fcf-a484-d519592de325/6ae9977e-919b-4292-b0e6-ff735491d0d2"
-					(reference "#PWR092")
+					(reference "#PWR077")
 					(unit 1)
 				)
@@
 		(dnp no)
 		(fields_autoplaced yes)
-		(property "Reference" "#PWR087"
+		(property "Reference" "#PWR072"
 			(at 67.945 49.53 0)
 			(effects
@@
 			(project "NHK2026_mainboard"
 				(path "/288b008e-4fe6-4fcf-a484-d519592de325/6ae9977e-919b-4292-b0e6-ff735491d0d2"
-					(reference "#PWR087")
+					(reference "#PWR072")
 					(unit 1)
 				)
@@
 		(dnp no)
 		(fields_autoplaced yes)
-		(property "Reference" "#PWR0100"
+		(property "Reference" "#PWR085"
 			(at 212.725 106.68 0)
 			(effects
@@
 			(project "NHK2026_mainboard"
 				(path "/288b008e-4fe6-4fcf-a484-d519592de325/6ae9977e-919b-4292-b0e6-ff735491d0d2"
-					(reference "#PWR0100")
+					(reference "#PWR085")
 					(unit 1)
 				)
@@
 		(dnp no)
 		(fields_autoplaced yes)
-		(property "Reference" "#PWR093"
+		(property "Reference" "#PWR078"
 			(at 156.845 138.43 0)
 			(effects
@@
 			(project "NHK2026_mainboard"
 				(path "/288b008e-4fe6-4fcf-a484-d519592de325/6ae9977e-919b-4292-b0e6-ff735491d0d2"
-					(reference "#PWR093")
+					(reference "#PWR078")
 					(unit 1)
 				)
@@
 		(dnp no)
 		(fields_autoplaced yes)
-		(property "Reference" "#PWR091"
+		(property "Reference" "#PWR076"
 			(at 100.965 106.68 0)
 			(effects
@@
 			(project "NHK2026_mainboard"
 				(path "/288b008e-4fe6-4fcf-a484-d519592de325/6ae9977e-919b-4292-b0e6-ff735491d0d2"
-					(reference "#PWR091")
+					(reference "#PWR076")
 					(unit 1)
 				)
@@
 		(dnp no)
 		(fields_autoplaced yes)
-		(property "Reference" "#PWR095"
+		(property "Reference" "#PWR080"
 			(at 158.115 68.58 0)
 			(effects
@@
 			(project "NHK2026_mainboard"
 				(path "/288b008e-4fe6-4fcf-a484-d519592de325/6ae9977e-919b-4292-b0e6-ff735491d0d2"
-					(reference "#PWR095")
+					(reference "#PWR080")
 					(unit 1)
 				)
@@
 		(dnp no)
 		(fields_autoplaced yes)
-		(property "Reference" "#PWR083"
+		(property "Reference" "#PWR068"
 			(at 45.085 121.92 0)
 			(effects
@@
 			(project "NHK2026_mainboard"
 				(path "/288b008e-4fe6-4fcf-a484-d519592de325/6ae9977e-919b-4292-b0e6-ff735491d0d2"
-					(reference "#PWR083")
+					(reference "#PWR068")
 					(unit 1)
 				)
@@
 		(dnp no)
 		(fields_autoplaced yes)
-		(property "Reference" "#PWR094"
+		(property "Reference" "#PWR079"
 			(at 158.115 50.8 0)
 			(effects
@@
 			(project "NHK2026_mainboard"
 				(path "/288b008e-4fe6-4fcf-a484-d519592de325/6ae9977e-919b-4292-b0e6-ff735491d0d2"
-					(reference "#PWR094")
+					(reference "#PWR079")
 					(unit 1)
 				)
@@
 		(dnp no)
 		(fields_autoplaced yes)
-		(property "Reference" "#PWR089"
+		(property "Reference" "#PWR074"
 			(at 67.945 99.06 0)
 			(effects
@@
 			(project "NHK2026_mainboard"
 				(path "/288b008e-4fe6-4fcf-a484-d519592de325/6ae9977e-919b-4292-b0e6-ff735491d0d2"
-					(reference "#PWR089")
+					(reference "#PWR074")
 					(unit 1)
 				)
@@
 		(dnp no)
 		(fields_autoplaced yes)
-		(property "Reference" "#PWR084"
+		(property "Reference" "#PWR069"
 			(at 45.085 138.43 0)
 			(effects
@@
 			(project "NHK2026_mainboard"
 				(path "/288b008e-4fe6-4fcf-a484-d519592de325/6ae9977e-919b-4292-b0e6-ff735491d0d2"
-					(reference "#PWR084")
+					(reference "#PWR069")
 					(unit 1)
 				)
@@
 		(dnp no)
 		(fields_autoplaced yes)
-		(property "Reference" "#PWR085"
+		(property "Reference" "#PWR070"
 			(at 46.355 50.8 0)
 			(effects
@@
 			(project "NHK2026_mainboard"
 				(path "/288b008e-4fe6-4fcf-a484-d519592de325/6ae9977e-919b-4292-b0e6-ff735491d0d2"
-					(reference "#PWR085")
+					(reference "#PWR070")
 					(unit 1)
 				)
@@
 		(dnp no)
 		(fields_autoplaced yes)
-		(property "Reference" "#PWR097"
+		(property "Reference" "#PWR082"
 			(at 179.705 88.9 0)
 			(effects
@@
 			(project "NHK2026_mainboard"
 				(path "/288b008e-4fe6-4fcf-a484-d519592de325/6ae9977e-919b-4292-b0e6-ff735491d0d2"
-					(reference "#PWR097")
+					(reference "#PWR082")
 					(unit 1)
 				)
@@
 		(dnp no)
 		(fields_autoplaced yes)
-		(property "Reference" "#PWR098"
+		(property "Reference" "#PWR083"
 			(at 179.705 99.06 0)
 			(effects
@@
 			(project "NHK2026_mainboard"
 				(path "/288b008e-4fe6-4fcf-a484-d519592de325/6ae9977e-919b-4292-b0e6-ff735491d0d2"
-					(reference "#PWR098")
+					(reference "#PWR083")
 					(unit 1)
 				)
@@
 		(dnp no)
 		(fields_autoplaced yes)
-		(property "Reference" "J29"
+		(property "Reference" "J14"
 			(at 109.855 86.3599 0)
 			(effects
@@
 			(project "NHK2026_mainboard"
 				(path "/288b008e-4fe6-4fcf-a484-d519592de325/6ae9977e-919b-4292-b0e6-ff735491d0d2"
-					(reference "J29")
+					(reference "J14")
 					(unit 1)
 				)
@@
 		(dnp no)
 		(fields_autoplaced yes)
-		(property "Reference" "#PWR099"
+		(property "Reference" "#PWR084"
 			(at 179.705 138.43 0)
 			(effects
@@
 			(project "NHK2026_mainboard"
 				(path "/288b008e-4fe6-4fcf-a484-d519592de325/6ae9977e-919b-4292-b0e6-ff735491d0d2"
-					(reference "#PWR099")
+					(reference "#PWR084")
 					(unit 1)
 				)
@@
 		(dnp no)
 		(fields_autoplaced yes)
-		(property "Reference" "#PWR090"
+		(property "Reference" "#PWR075"
 			(at 67.945 138.43 0)
 			(effects
@@
 			(project "NHK2026_mainboard"
 				(path "/288b008e-4fe6-4fcf-a484-d519592de325/6ae9977e-919b-4292-b0e6-ff735491d0d2"
-					(reference "#PWR090")
-					(unit 1)
-				)
+					(reference "#PWR075")
+					(unit 1)
+				)

Commit message: メイン基板完成
Parts:
- renumbered R25 to R27, R26 to R28, R27 to R29, R28 to R30, R29 to R31, R30 to R32, R31 to R33, R32 to R34, R33 to R35, R34 to R36, R35 to R37, R36 to R38

Commit message: 微修正
Parts:
- renumbered C15 to C21, C16 to C22, C17 to C23, C18 to C24
Changed lines of the file:
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@@
 		(dnp no)
 		(fields_autoplaced yes)
-		(property "Reference" "C18"
+		(property "Reference" "C24"
 			(at 161.036 53.9663 0)
 			(effects
@@
 			(project "NHK2026_mainboard"
 				(path "/288b008e-4fe6-4fcf-a484-d519592de325/6ae9977e-919b-4292-b0e6-ff735491d0d2"
-					(reference "C18")
+					(reference "C24")
 					(unit 1)
 				)
@@
 		(dnp no)
 		(fields_autoplaced yes)
-		(property "Reference" "#PWR076"
+		(property "Reference" "#PWR088"
 			(at 67.945 88.9 0)
 			(effects
@@
 			(project "NHK2026_mainboard"
 				(path "/288b008e-4fe6-4fcf-a484-d519592de325/6ae9977e-919b-4292-b0e6-ff735491d0d2"
-					(reference "#PWR076")
+					(reference "#PWR088")
 					(unit 1)
 				)
@@
 		(dnp no)
 		(fields_autoplaced yes)
-		(property "Reference" "#PWR084"
+		(property "Reference" "#PWR096"
 			(at 179.705 49.53 0)
 			(effects
@@
 			(project "NHK2026_mainboard"
 				(path "/288b008e-4fe6-4fcf-a484-d519592de325/6ae9977e-919b-4292-b0e6-ff735491d0d2"
-					(reference "#PWR084")
+					(reference "#PWR096")
 					(unit 1)
 				)
@@
 		(dnp no)
 		(fields_autoplaced yes)
-		(property "Reference" "#PWR074"
+		(property "Reference" "#PWR086"
 			(at 46.355 68.58 0)
 			(effects
@@
 			(project "NHK2026_mainboard"
 				(path "/288b008e-4fe6-4fcf-a484-d519592de325/6ae9977e-919b-4292-b0e6-ff735491d0d2"
-					(reference "#PWR074")
+					(reference "#PWR086")
 					(unit 1)
 				)
@@
 		(dnp no)
 		(fields_autoplaced yes)
-		(property "Reference" "#PWR080"
+		(property "Reference" "#PWR092"
 			(at 156.845 121.92 0)
 			(effects
@@
 			(project "NHK2026_mainboard"
 				(path "/288b008e-4fe6-4fcf-a484-d519592de325/6ae9977e-919b-4292-b0e6-ff735491d0d2"
-					(reference "#PWR080")
+					(reference "#PWR092")
 					(unit 1)
 				)
@@
 		(dnp no)
 		(fields_autoplaced yes)
-		(property "Reference" "#PWR075"
+		(property "Reference" "#PWR087"
 			(at 67.945 49.53 0)
 			(effects
@@
 			(project "NHK2026_mainboard"
 				(path "/288b008e-4fe6-4fcf-a484-d519592de325/6ae9977e-919b-4292-b0e6-ff735491d0d2"
-					(reference "#PWR075")
+					(reference "#PWR087")
 					(unit 1)
 				)
@@
 		(dnp no)
 		(fields_autoplaced yes)
-		(property "Reference" "#PWR088"
+		(property "Reference" "#PWR0100"
 			(at 212.725 106.68 0)
 			(effects
@@
 			(project "NHK2026_mainboard"
 				(path "/288b008e-4fe6-4fcf-a484-d519592de325/6ae9977e-919b-4292-b0e6-ff735491d0d2"
-					(reference "#PWR088")
+					(reference "#PWR0100")
 					(unit 1)
 				)
@@
 		(dnp no)
 		(fields_autoplaced yes)
-		(property "Reference" "#PWR081"
+		(property "Reference" "#PWR093"
 			(at 156.845 138.43 0)
 			(effects
@@
 			(project "NHK2026_mainboard"
 				(path "/288b008e-4fe6-4fcf-a484-d519592de325/6ae9977e-919b-4292-b0e6-ff735491d0d2"
-					(reference "#PWR081")
+					(reference "#PWR093")
 					(unit 1)
 				)
@@
 		(dnp no)
 		(fields_autoplaced yes)
-		(property "Reference" "#PWR079"
+		(property "Reference" "#PWR091"
 			(at 100.965 106.68 0)
 			(effects
@@
 			(project "NHK2026_mainboard"
 				(path "/288b008e-4fe6-4fcf-a484-d519592de325/6ae9977e-919b-4292-b0e6-ff735491d0d2"
-					(reference "#PWR079")
+					(reference "#PWR091")
 					(unit 1)
 				)
@@
 		(dnp no)
 		(fields_autoplaced yes)
-		(property "Reference" "#PWR083"
+		(property "Reference" "#PWR095"
 			(at 158.115 68.58 0)
 			(effects
@@
 			(project "NHK2026_mainboard"
 				(path "/288b008e-4fe6-4fcf-a484-d519592de325/6ae9977e-919b-4292-b0e6-ff735491d0d2"
-					(reference "#PWR083")
+					(reference "#PWR095")
 					(unit 1)
 				)
@@
 		(dnp no)
 		(fields_autoplaced yes)
-		(property "Reference" "C16"
+		(property "Reference" "C22"
 			(at 49.276 53.9663 0)
 			(effects
@@
 			(project "NHK2026_mainboard"
 				(path "/288b008e-4fe6-4fcf-a484-d519592de325/6ae9977e-919b-4292-b0e6-ff735491d0d2"
-					(reference "C16")
+					(reference "C22")
 					(unit 1)
 				)
@@
 		(dnp no)
 		(fields_autoplaced yes)
-		(property "Reference" "#PWR071"
+		(property "Reference" "#PWR083"
 			(at 45.085 121.92 0)
 			(effects
@@
 			(project "NHK2026_mainboard"
 				(path "/288b008e-4fe6-4fcf-a484-d519592de325/6ae9977e-919b-4292-b0e6-ff735491d0d2"
-					(reference "#PWR071")
+					(reference "#PWR083")
 					(unit 1)
 				)
@@
 		(dnp no)
 		(fields_autoplaced yes)
-		(property "Reference" "#PWR082"
+		(property "Reference" "#PWR094"
 			(at 158.115 50.8 0)
 			(effects
@@
 			(project "NHK2026_mainboard"
 				(path "/288b008e-4fe6-4fcf-a484-d519592de325/6ae9977e-919b-4292-b0e6-ff735491d0d2"
-					(reference "#PWR082")
+					(reference "#PWR094")
 					(unit 1)
 				)
@@
 		(dnp no)
 		(fields_autoplaced yes)
-		(property "Reference" "#PWR077"
+		(property "Reference" "#PWR089"
 			(at 67.945 99.06 0)
 			(effects
@@
 			(project "NHK2026_mainboard"
 				(path "/288b008e-4fe6-4fcf-a484-d519592de325/6ae9977e-919b-4292-b0e6-ff735491d0d2"
-					(reference "#PWR077")
+					(reference "#PWR089")
 					(unit 1)
 				)
@@
 		(dnp no)
 		(fields_autoplaced yes)
-		(property "Reference" "#PWR072"
+		(property "Reference" "#PWR084"
 			(at 45.085 138.43 0)
 			(effects
@@
 			(project "NHK2026_mainboard"
 				(path "/288b008e-4fe6-4fcf-a484-d519592de325/6ae9977e-919b-4292-b0e6-ff735491d0d2"
-					(reference "#PWR072")
+					(reference "#PWR084")
 					(unit 1)
 				)
@@
 		(dnp no)
 		(fields_autoplaced yes)
-		(property "Reference" "#PWR073"
+		(property "Reference" "#PWR085"
 			(at 46.355 50.8 0)
 			(effects
@@
 			(project "NHK2026_mainboard"
 				(path "/288b008e-4fe6-4fcf-a484-d519592de325/6ae9977e-919b-4292-b0e6-ff735491d0d2"
-					(reference "#PWR073")
+					(reference "#PWR085")
 					(unit 1)
 				)
@@
 		(on_board yes)
 		(dnp no)
-		(property "Reference" "C17"
+		(property "Reference" "C23"
 			(at 160.655 123.19 0)
 			(effects
@@
 			(project "NHK2026_mainboard"
 				(path "/288b008e-4fe6-4fcf-a484-d519592de325/6ae9977e-919b-4292-b0e6-ff735491d0d2"
-					(reference "C17")
+					(reference "C23")
 					(unit 1)
 				)
@@
 		(dnp no)
 		(fields_autoplaced yes)
-		(property "Reference" "#PWR085"
+		(property "Reference" "#PWR097"
 			(at 179.705 88.9 0)
 			(effects
@@
 			(project "NHK2026_mainboard"
 				(path "/288b008e-4fe6-4fcf-a484-d519592de325/6ae9977e-919b-4292-b0e6-ff735491d0d2"
-					(reference "#PWR085")
+					(reference "#PWR097")
 					(unit 1)
 				)
@@
 		(dnp no)
 		(fields_autoplaced yes)
-		(property "Reference" "#PWR086"
+		(property "Reference" "#PWR098"
 			(at 179.705 99.06 0)
 			(effects
@@
 			(project "NHK2026_mainboard"
 				(path "/288b008e-4fe6-4fcf-a484-d519592de325/6ae9977e-919b-4292-b0e6-ff735491d0d2"
-					(reference "#PWR086")
+					(reference "#PWR098")
 					(unit 1)
 				)
@@
 		(on_board yes)
 		(dnp no)
-		(property "Reference" "C15"
+		(property "Reference" "C21"
 			(at 48.895 123.19 0)
 			(effects
@@
 			(project "NHK2026_mainboard"
 				(path "/288b008e-4fe6-4fcf-a484-d519592de325/6ae9977e-919b-4292-b0e6-ff735491d0d2"
-					(reference "C15")
+					(reference "C21")
 					(unit 1)
 				)
@@
 		(dnp no)
 		(fields_autoplaced yes)
-		(property "Reference" "#PWR087"
+		(property "Reference" "#PWR099"
 			(at 179.705 138.43 0)
 			(effects
@@
 			(project "NHK2026_mainboard"
 				(path "/288b008e-4fe6-4fcf-a484-d519592de325/6ae9977e-919b-4292-b0e6-ff735491d0d2"
-					(reference "#PWR087")
+					(reference "#PWR099")
 					(unit 1)
 				)
@@
 		(dnp no)
 		(fields_autoplaced yes)
-		(property "Reference" "#PWR078"
+		(property "Reference" "#PWR090"
 			(at 67.945 138.43 0)
 			(effects
@@
 			(project "NHK2026_mainboard"
 				(path "/288b008e-4fe6-4fcf-a484-d519592de325/6ae9977e-919b-4292-b0e6-ff735491d0d2"
-					(reference "#PWR078")
-					(unit 1)
-				)
+					(reference "#PWR090")
+					(unit 1)
+				)
