File: wtt12l.kicad_sch (KiCad schematic)
At the start: 18 parts

Commit message: 回路図だいたい完成
Parts:
- gave numbers to parts that had none: 18

Commit message: 何こっち見てんだよ
Parts:
- J33: renamed from J40; footprint (none) -> Connector_JST:JST_XH_B4B-XH-A_1x04_P2.50mm_Vertical
- J34: renamed from J41; footprint (none) -> Connector_JST:JST_XH_B4B-XH-A_1x04_P2.50mm_Vertical
- J35: renamed from J42; footprint (none) -> Connector_JST:JST_XH_B4B-XH-A_1x04_P2.50mm_Vertical
- R39: renamed from R38; footprint (none) -> Resistor_SMD:R_0603_1608Metric_Pad0.98x0.95mm_HandSolder
- R40: renamed from R39; footprint (none) -> Resistor_SMD:R_0603_1608Metric_Pad0.98x0.95mm_HandSolder
- R41: renamed from R40; footprint (none) -> Resistor_SMD:R_0603_1608Metric_Pad0.98x0.95mm_HandSolder
- R42: renamed from R41; footprint (none) -> Resistor_SMD:R_0603_1608Metric_Pad0.98x0.95mm_HandSolder
- R43: renamed from R42; footprint (none) -> Resistor_SMD:R_0603_1608Metric_Pad0.98x0.95mm_HandSolder
- R44: renamed from R43; footprint (none) -> Resistor_SMD:R_0603_1608Metric_Pad0.98x0.95mm_HandSolder
- R45: renamed from R44; footprint (none) -> Resistor_SMD:R_0603_1608Metric_Pad0.98x0.95mm_HandSolder
- R46: renamed from R45; footprint (none) -> Resistor_SMD:R_0603_1608Metric_Pad0.98x0.95mm_HandSolder
- R47: renamed from R46; footprint (none) -> Resistor_SMD:R_0603_1608Metric_Pad0.98x0.95mm_HandSolder
- R48: renamed from R47; footprint (none) -> Resistor_SMD:R_0603_1608Metric_Pad0.98x0.95mm_HandSolder
- R49: renamed from R48; footprint (none) -> Resistor_SMD:R_0603_1608Metric_Pad0.98x0.95mm_HandSolder
- R50: renamed from R49; footprint (none) -> Resistor_SMD:R_0603_1608Metric_Pad0.98x0.95mm_HandSolder
- renumbered C22 to C23, C23 to C24, C24 to C25

Commit message: 配線だいたい完了
Parts:
- renumbered J33 to J18, J34 to J19, J35 to J20
Changed lines of the file:
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@@
 		(dnp no)
 		(fields_autoplaced yes)
-		(property "Reference" "#PWR0132"
+		(property "Reference" "#PWR0117"
 			(at 254 73.66 0)
 			(effects
@@
 			(project "NHK2026_mainboard"
 				(path "/288b008e-4fe6-4fcf-a484-d519592de325/6646f01f-a2b4-4ddb-9fd5-82c7b2d7f873"
-					(reference "#PWR0132")
+					(reference "#PWR0117")
 					(unit 1)
 				)
@@
 		(dnp no)
 		(fields_autoplaced yes)
-		(property "Reference" "#PWR0117"
+		(property "Reference" "#PWR0102"
 			(at 80.01 36.83 0)
 			(effects
@@
 			(project "NHK2026_mainboard"
 				(path "/288b008e-4fe6-4fcf-a484-d519592de325/6646f01f-a2b4-4ddb-9fd5-82c7b2d7f873"
-					(reference "#PWR0117")
+					(reference "#PWR0102")
 					(unit 1)
 				)
@@
 		(dnp no)
 		(fields_autoplaced yes)
-		(property "Reference" "#PWR0122"
+		(property "Reference" "#PWR0107"
 			(at 151.13 73.66 0)
 			(effects
@@
 			(project "NHK2026_mainboard"
 				(path "/288b008e-4fe6-4fcf-a484-d519592de325/6646f01f-a2b4-4ddb-9fd5-82c7b2d7f873"
-					(reference "#PWR0122")
+					(reference "#PWR0107")
 					(unit 1)
 				)
@@
 		(dnp no)
 		(fields_autoplaced yes)
-		(property "Reference" "#PWR0119"
+		(property "Reference" "#PWR0104"
 			(at 87.63 57.15 0)
 			(effects
@@
 			(project "NHK2026_mainboard"
 				(path "/288b008e-4fe6-4fcf-a484-d519592de325/6646f01f-a2b4-4ddb-9fd5-82c7b2d7f873"
-					(reference "#PWR0119")
+					(reference "#PWR0104")
 					(unit 1)
 				)
@@
 		(dnp no)
 		(fields_autoplaced yes)
-		(property "Reference" "J35"
+		(property "Reference" "J20"
 			(at 255.27 39.3699 0)
 			(effects
@@
 			(project "NHK2026_mainboard"
 				(path "/288b008e-4fe6-4fcf-a484-d519592de325/6646f01f-a2b4-4ddb-9fd5-82c7b2d7f873"
-					(reference "J35")
+					(reference "J20")
 					(unit 1)
 				)
@@
 		(dnp no)
 		(fields_autoplaced yes)
-		(property "Reference" "#PWR0116"
+		(property "Reference" "#PWR0101"
 			(at 68.58 73.66 0)
 			(effects
@@
 			(project "NHK2026_mainboard"
 				(path "/288b008e-4fe6-4fcf-a484-d519592de325/6646f01f-a2b4-4ddb-9fd5-82c7b2d7f873"
-					(reference "#PWR0116")
+					(reference "#PWR0101")
 					(unit 1)
 				)
@@
 		(dnp no)
 		(fields_autoplaced yes)
-		(property "Reference" "J34"
+		(property "Reference" "J19"
 			(at 171.45 39.3699 0)
 			(effects
@@
 			(project "NHK2026_mainboard"
 				(path "/288b008e-4fe6-4fcf-a484-d519592de325/6646f01f-a2b4-4ddb-9fd5-82c7b2d7f873"
-					(reference "J34")
+					(reference "J19")
 					(unit 1)
 				)
@@
 		(dnp no)
 		(fields_autoplaced yes)
-		(property "Reference" "#PWR0120"
+		(property "Reference" "#PWR0105"
 			(at 87.63 73.66 0)
 			(effects
@@
 			(project "NHK2026_mainboard"
 				(path "/288b008e-4fe6-4fcf-a484-d519592de325/6646f01f-a2b4-4ddb-9fd5-82c7b2d7f873"
-					(reference "#PWR0120")
+					(reference "#PWR0105")
 					(unit 1)
 				)
@@
 		(dnp no)
 		(fields_autoplaced yes)
-		(property "Reference" "#PWR0118"
+		(property "Reference" "#PWR0103"
 			(at 80.01 53.34 0)
 			(effects
@@
 			(project "NHK2026_mainboard"
 				(path "/288b008e-4fe6-4fcf-a484-d519592de325/6646f01f-a2b4-4ddb-9fd5-82c7b2d7f873"
-					(reference "#PWR0118")
+					(reference "#PWR0103")
 					(unit 1)
 				)
@@
 		(dnp no)
 		(fields_autoplaced yes)
-		(property "Reference" "#PWR0115"
+		(property "Reference" "#PWR0100"
 			(at 41.91 73.66 0)
 			(effects
@@
 			(project "NHK2026_mainboard"
 				(path "/288b008e-4fe6-4fcf-a484-d519592de325/6646f01f-a2b4-4ddb-9fd5-82c7b2d7f873"
-					(reference "#PWR0115")
+					(reference "#PWR0100")
 					(unit 1)
 				)
@@
 		(dnp no)
 		(fields_autoplaced yes)
-		(property "Reference" "#PWR0126"
+		(property "Reference" "#PWR0111"
 			(at 170.18 73.66 0)
 			(effects
@@
 			(project "NHK2026_mainboard"
 				(path "/288b008e-4fe6-4fcf-a484-d519592de325/6646f01f-a2b4-4ddb-9fd5-82c7b2d7f873"
-					(reference "#PWR0126")
+					(reference "#PWR0111")
 					(unit 1)
 				)
@@
 		(dnp no)
 		(fields_autoplaced yes)
-		(property "Reference" "#PWR0127"
+		(property "Reference" "#PWR0112"
 			(at 208.28 73.66 0)
 			(effects
@@
 			(project "NHK2026_mainboard"
 				(path "/288b008e-4fe6-4fcf-a484-d519592de325/6646f01f-a2b4-4ddb-9fd5-82c7b2d7f873"
-					(reference "#PWR0127")
+					(reference "#PWR0112")
 					(unit 1)
 				)
@@
 		(dnp no)
 		(fields_autoplaced yes)
-		(property "Reference" "#PWR0131"
+		(property "Reference" "#PWR0116"
 			(at 254 57.15 0)
 			(effects
@@
 			(project "NHK2026_mainboard"
 				(path "/288b008e-4fe6-4fcf-a484-d519592de325/6646f01f-a2b4-4ddb-9fd5-82c7b2d7f873"
-					(reference "#PWR0131")
+					(reference "#PWR0116")
 					(unit 1)
 				)
@@
 		(dnp no)
 		(fields_autoplaced yes)
-		(property "Reference" "#PWR0121"
+		(property "Reference" "#PWR0106"
 			(at 124.46 73.66 0)
 			(effects
@@
 			(project "NHK2026_mainboard"
 				(path "/288b008e-4fe6-4fcf-a484-d519592de325/6646f01f-a2b4-4ddb-9fd5-82c7b2d7f873"
-					(reference "#PWR0121")
+					(reference "#PWR0106")
 					(unit 1)
 				)
@@
 		(dnp no)
 		(fields_autoplaced yes)
-		(property "Reference" "#PWR0128"
+		(property "Reference" "#PWR0113"
 			(at 234.95 73.66 0)
 			(effects
@@
 			(project "NHK2026_mainboard"
 				(path "/288b008e-4fe6-4fcf-a484-d519592de325/6646f01f-a2b4-4ddb-9fd5-82c7b2d7f873"
-					(reference "#PWR0128")
+					(reference "#PWR0113")
 					(unit 1)
 				)
@@
 		(dnp no)
 		(fields_autoplaced yes)
-		(property "Reference" "#PWR0129"
+		(property "Reference" "#PWR0114"
 			(at 246.38 36.83 0)
 			(effects
@@
 			(project "NHK2026_mainboard"
 				(path "/288b008e-4fe6-4fcf-a484-d519592de325/6646f01f-a2b4-4ddb-9fd5-82c7b2d7f873"
-					(reference "#PWR0129")
+					(reference "#PWR0114")
 					(unit 1)
 				)
@@
 		(dnp no)
 		(fields_autoplaced yes)
-		(property "Reference" "#PWR0123"
+		(property "Reference" "#PWR0108"
 			(at 162.56 36.83 0)
 			(effects
@@
 			(project "NHK2026_mainboard"
 				(path "/288b008e-4fe6-4fcf-a484-d519592de325/6646f01f-a2b4-4ddb-9fd5-82c7b2d7f873"
-					(reference "#PWR0123")
+					(reference "#PWR0108")
 					(unit 1)
 				)
@@
 		(dnp no)
 		(fields_autoplaced yes)
-		(property "Reference" "#PWR0125"
+		(property "Reference" "#PWR0110"
 			(at 170.18 57.15 0)
 			(effects
@@
 			(project "NHK2026_mainboard"
 				(path "/288b008e-4fe6-4fcf-a484-d519592de325/6646f01f-a2b4-4ddb-9fd5-82c7b2d7f873"
-					(reference "#PWR0125")
+					(reference "#PWR0110")
 					(unit 1)
 				)
@@
 		(dnp no)
 		(fields_autoplaced yes)
-		(property "Reference" "#PWR0130"
+		(property "Reference" "#PWR0115"
 			(at 246.38 53.34 0)
 			(effects
@@
 			(project "NHK2026_mainboard"
 				(path "/288b008e-4fe6-4fcf-a484-d519592de325/6646f01f-a2b4-4ddb-9fd5-82c7b2d7f873"
-					(reference "#PWR0130")
+					(reference "#PWR0115")
 					(unit 1)
 				)
@@
 		(dnp no)
 		(fields_autoplaced yes)
-		(property "Reference" "J33"
+		(property "Reference" "J18"
 			(at 88.9 39.3699 0)
 			(effects
@@
 			(project "NHK2026_mainboard"
 				(path "/288b008e-4fe6-4fcf-a484-d519592de325/6646f01f-a2b4-4ddb-9fd5-82c7b2d7f873"
-					(reference "J33")
+					(reference "J18")
 					(unit 1)
 				)
@@
 		(dnp no)
 		(fields_autoplaced yes)
-		(property "Reference" "#PWR0124"
+		(property "Reference" "#PWR0109"
 			(at 162.56 53.34 0)
 			(effects
@@
 			(project "NHK2026_mainboard"
 				(path "/288b008e-4fe6-4fcf-a484-d519592de325/6646f01f-a2b4-4ddb-9fd5-82c7b2d7f873"
-					(reference "#PWR0124")
-					(unit 1)
-				)
+					(reference "#PWR0109")
+					(unit 1)
+				)

Commit message: メイン基板完成
Parts:
- renumbered R39 to R41, R40 to R42, R41 to R43, R42 to R44, R43 to R45, R44 to R46, R45 to R47, R46 to R48, R47 to R49, R48 to R50, R49 to R51, R50 to R52

Commit message: 微修正
Parts:
- added C30: 25V 470u, Capacitor_THT:CP_Radial_D8.0mm_P3.50mm, symbol Device:C_Polarized
- renumbered C23 to C29, C24 to C31, C25 to C32
Connections:
- net +12V: now also C30.1
- net GND: now also C30.2
